File: hardware/schematics/Motor_Driver/Motor_Driver/Motor_Driver.sch (KiCad schematic (older format))
At the start: 28 parts, among them J1 Screw_Terminal_01x04, J2 Screw_Terminal_01x02, J3 Screw_Terminal_01x02, J4 Screw_Terminal_01x03, J5 Screw_Terminal_01x02, J6 Screw_Terminal_01x02, J7 Screw_Terminal_01x01, J8 Screw_Terminal_01x01, U1 ATmega328P-PU, U2 LM78M05_TO220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

Commit message: schematic mainboard satart
Parts:
- added C?: CP, symbol Device:CP
- added D? (x8): D, symbol Device:D
- added J? (x3): Screw_Terminal_01x02, symbol Connector:Screw_Terminal_01x02
- added J?: Screw_Terminal_01x04, symbol Connector:Screw_Terminal_01x04
- added M? (x4): Motor_DC, symbol Motor:Motor_DC
- added U? (x3): HC-SR04, symbol robot:HC-SR04
- added U?: L298HN, Package_TO_SOT_THT:TO-220-15_P2.54x2.54mm_StaggerOdd_Lead4.58mm_Vertical, symbol Driver_Motor:L298HN
Connections:
- net GND: now also U?.1 (SENSE_A), U?.8 (GND)
- new net: J?.1 (Pin_1), U?.10 (IN3)
- new net: J?.1 (Pin_1), U?.11 (EnB)
- new net: J?.2 (Pin_2), U?.12 (IN4)
- new net: D?.1 (K), D?.2 (A), J?.1 (Pin_1), U?.13 (OUT3)
- new net: D?.1 (K), D?.2 (A), J?.2 (Pin_2), U?.14 (OUT4)
- new net: D?.1 (K), D?.2 (A), J?.1 (Pin_1), U?.2 (OUT1)
- new net: D?.1 (K), D?.2 (A), J?.2 (Pin_2), U?.3 (OUT2)
- new net: C?.1, D?.1 (K), D?.1 (K), D?.1 (K), D?.1 (K), U?.4 (Vs)
- new net: J?.4 (Pin_4), U?.5 (IN1)
- new net: J?.2 (Pin_2), U?.6 (EnA)
- new net: J?.3 (Pin_3), U?.7 (IN2)
- new net: C?.2, D?.2 (A), D?.2 (A), D?.2 (A), D?.2 (A)
Other:
- moved on the sheet: C1, C2, C3, C4, C5, D1, D2, D3, D4, D5, D6, D7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
