File: hardware/schematics/TestScheme/TestScheme.kicad_pcb (KiCad board)
At the start: 2 copper layers, 50 x 50 mm, 4 parts, among them J1 Screw_Terminal_01x02, SW1 SW_DIP_x01

Commit message: obstacle detection
Other:
- net class Default removed
